File: loraine/node_hw/loraine_node.kicad_pcb (KiCad board)
At the start: 2 copper layers, 50.8 x 53.3 mm, 41 parts, among them CON1 BARREL_JACK, IC1 ATTINY2313A-S, P1 MOLEX, P2 MOLEX, P3 SOLDER_PAD, P4 ICSP, P5 OUTPUTS, P6 BUS, P7 BUS_THRU, Q1 BD679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

Commit message: Added locking 2-way MOLEX headers
MOLEX part 22-23-2021 for header = farnell 1462926
MOLEX part 22-01-3027 for receptacle = farnell 1462825
Parts:
- P1: value MOLEX -> POWER_THRU; footprint Connect:SIL-2 -> molex-22-23-2021:SIL-2
- P2: value MOLEX -> POWER; footprint Connect:SIL-2 -> molex-22-23-2021:SIL-2
- P6, P7: footprint Connect:SIL-2 -> molex-22-23-2021:SIL-2

Commit message: Added proper solder pad footprint
Parts:
- P3: footprint Connect:SIL-2 -> solder_pad:SIL-2
- moved P3 7.11 mm to (92.9, 114.1)

Commit message: Improved power solder pad
Added strain relief, made pin 1 (negative) rectangular
Parts:
- moved P3 1.93 mm to (94.6, 115.1)
