File: loraine/hardware/loraine_node.kicad_pcb (KiCad board)
At the start: 2 copper layers, 50.8 x 53.3 mm, 41 parts, among them CON1 BARREL_JACK, IC1 ATTINY2313A-S, P1 POWER_THRU, P2 POWER, P3 SOLDER_PAD, P4 ICSP, P5 OUTPUTS, P6 BUS, P7 BUS_THRU, Q1 BD679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

Commit message: Changed LED component/footprint to single colour  devices
Parts:
- added D2: GREEN, power_led:power_led, F.Cu at (52.5, 111.7)
- added D3: BLUE, power_led:power_led, F.Cu at (111.7, 107.2)
- D1: value STAR_LED -> RED; footprint led_module:led_module -> power_led:power_led
Connections:
- D1 pad 3: Net-(D1-Pad3) -> (no net)
- R1 pad 1: Net-(D1-Pad6) -> Net-(D1-Pad2)
- R2 pad 1: Net-(D1-Pad5) -> Net-(D2-Pad2)
- R3 pad 1: Net-(D1-Pad4) -> Net-(D3-Pad2)
- U3 pad 4: Net-(D1-Pad4) -> Net-(D3-Pad2)
- U3 pad 6: Net-(D1-Pad3) -> Net-(D3-Pad1)
- U4 pad 4: Net-(D1-Pad5) -> Net-(D2-Pad2)
- U4 pad 6: Net-(D1-Pad2) -> Net-(D2-Pad1)
- U5 pad 4: Net-(D1-Pad6) -> Net-(D1-Pad2)
