File: loraine/hardware/loraine_node.kicad_pcb (KiCad board)
At the start: 2 copper layers, 50.8 x 53.3 mm, 41 parts, among them CON1 BARREL_JACK, IC1 ATTINY2313A-S, P1 POWER_THRU, P2 POWER, P3 SOLDER_PAD, P4 ICSP, P5 OUTPUTS, P6 BUS, P7 BUS_THRU, Q1 BD679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

Commit message: Heatsunk LED footprint and board pads
Parts:
- D1: footprint led_module:led_module -> heatsunk_star_led:heatsunk_star_led_board
- moved D1 52.5 mm to (125.3, 100.9)
