File: loraine/hardware/loraine_node.sch (KiCad schematic (older format))
At the start: 41 parts, among them CON1 BARREL_JACK, IC1 ATTINY2313A-S, P1 POWER_THRU, P2 POWER, P3 SOLDER_PAD, P4 ICSP, P5 OUTPUTS, P6 BUS, P7 BUS_THRU, Q1 BD679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

Commit message: Changed LED component/footprint to single colour  devices
Parts:
- removed D1: STAR_LED, symbol STAR_LED
- added D1: RED, symbol LED
- added D2: GREEN, symbol LED
- added D3: BLUE, symbol LED
Connections:
- net at R3.1, U3.4 (REF): now also D3.2 (K)
- net at U3.6 (Q): now also D3.1 (A)
- net at R2.1, U4.4 (REF): now also D2.2 (K)
- net at U4.6 (Q): now also D2.1 (A)
- net at R1.1, U5.4 (REF): now also D1.2 (K)
- net at U5.6 (Q): now also D1.1 (A)
Changed lines of the file:
@@
 Connection ~ 10400 4550
 Wire Wire Line
-	10400 4400 10400 4900
+	10400 4325 10400 4900
 Wire Wire Line
 	10400 5400 10400 5650
-$Comp
-L STAR_LED D1
-U 1 1 53619F29
-P 10400 4150
-F 0 "D1" V 10000 4150 50  0000 C CNN
-F 1 "STAR_LED" V 10750 4200 50  0000 C CNN
-F 2 "" V 10200 4050 60  0000 C CNN
-F 3 "" V 10200 4050 60  0000 C CNN
-	1    10400 4150
-	1    0    0    -1
-$EndComp
 Wire Wire Line
-	10200 4400 10200 4800
+	10200 4325 10200 4800
 Connection ~ 10200 4500
 Wire Wire Line
 	8300 4600 10600 4600
 Wire Wire Line
-	10600 4400 10600 4800
+	10600 4325 10600 4800
 Connection ~ 10600 4600
 Wire Wire Line
-	10400 2800 10400 3850
+	10400 2800 10400 3925
 Wire Wire Line
-	10600 1650 10600 3850
+	10600 1650 10600 3925
 Wire Wire Line
 	9450 1650 10600 1650
@@
 Wire Wire Line
 	3500 3200 3450 3200
+$Comp
+L LED D1
+U 1 1 536C1D22
+P 10200 4125
+F 0 "D1" H 10400 4050 50  0000 C CNN
+F 1 "RED" H 10200 4025 50  0000 C CNN
+F 2 "" H 10200 4125 60  0000 C CNN
+F 3 "" H 10200 4125 60  0000 C CNN
+	1    10200 4125
+	0    1    1    0
+$EndComp
+$Comp
+L LED D2
+U 1 1 536C1D80
+P 10400 4125
+F 0 "D2" H 10600 4050 50  0000 C CNN
+F 1 "GREEN" H 10375 4025 50  0000 C CNN
+F 2 "" H 10400 4125 60  0000 C CNN
+F 3 "" H 10400 4125 60  0000 C CNN
+	1    10400 4125
+	0    1    1    0
+$EndComp
+$Comp
+L LED D3
+U 1 1 536C1DC9
+P 10600 4125
+F 0 "D3" H 10800 4050 50  0000 C CNN
+F 1 "BLUE" H 10575 4025 50  0000 C CNN
+F 2 "" H 10600 4125 60  0000 C CNN
+F 3 "" H 10600 4125 60  0000 C CNN
+	1    10600 4125
+	0    1    1    0
+$EndComp
+Wire Wire Line
+	10200 3850 10200 3925
 $EndSCHEMATC
