File: loraine/hardware/uplighter/uplighter.kicad_pcb (KiCad board)
At the start: 2 copper layers, 10 parts, among them P1 CONN_9, U1 TL4242, U2 TL4242, U3 TL4242

Commit message: Split board-board connector to 3x SIL3
Parts:
- removed P1: CONN_9, Connect:SIL-9
- added K1: CONN_GND, Connect:SIL-3, F.Cu at (110.2, 110.5)
- added K2: CONN_LEDS, Connect:SIL-3, F.Cu at (109.7, 115.4)
- added K3: CONN_12V, Connect:SIL-3, F.Cu at (109.9, 120.8)
