File: loraine/hardware/uplighter/uplighter.kicad_pcb (KiCad board)
At the start: 2 copper layers, 50 x 50 mm, 17 parts, among them CON1 BARREL_JACK, K1 CONN_3, K2 CONN_3, K3 CONN_3, P1 POWER_THRU, P2 POWER, P3 SOLDER_PAD, U1 TL4242, U2 TL4242, U3 TL4242

Commit message: Nominally finished both PCBs
Parts:
- added G***: LOGO, hypnospiral:hypnospiral_lessbig, B.Cu at (124.3, 124.7)
- R1, R2, R3: value R -> 1R2
- moved CON1 1.89 mm to (105.8, 145.8)
Connections:
- CON1 pad 3: (no net) -> GND
- U1 pad 2: (no net) -> Net-(U1-Pad2)
- U1 pad 5: (no net) -> Net-(U1-Pad5)
- U1 pad 7: (no net) -> Net-(U1-Pad7)
- U2 pad 2: (no net) -> Net-(U2-Pad2)
- U2 pad 5: (no net) -> Net-(U2-Pad5)
- U2 pad 7: (no net) -> Net-(U2-Pad7)
- U3 pad 2: (no net) -> Net-(U3-Pad2)
- U3 pad 5: (no net) -> Net-(U3-Pad5)
- U3 pad 7: (no net) -> Net-(U3-Pad7)
Routing:
- net GND: track 225.5 -> 205.8 mm, vias 41 -> 26
- net +5V: track 186.9 -> 179.7 mm
Other:
- board text added: "+"
- board text added: "+5V"
- board text added: "2014-07-28"
- board text added: "B+"
- board text added: "B-"
- board text added: "BLUE"
- board text added: "DATA"
- board text added: "DAVID TURNER ADAM GREIG"
- board text added: "G+"
- board text added: "G-"
- board text added: "GND"
- board text added: "GREEN"
- board text added: "LORAINE"
- board text added: "LORAINE UPLIGHTER"
- board text added: "R+"
- board text added: "R-"
- board text added: "RED"
- board text added: "UPLIGHTER"
- board text added: "r1"
