File: loraine/hardware/uplighter/uplighter.sch (KiCad schematic (older format))
At the start: 10 parts, among them P1 CONN_9, U1 TL4242, U2 TL4242, U3 TL4242

Commit message: Split board-board connector to 3x SIL3
Parts:
- removed P1: CONN_9, symbol CONN_9
- added K1: CONN_GND, symbol CONN_3
- added K2: CONN_LEDS, symbol CONN_3
- added K3: CONN_12V, symbol CONN_3
Changed lines of the file:
@@
 LIBS:valves
 LIBS:tl4242
+LIBS:uplighter-cache
 EELAYER 24 0
 EELAYER END
@@
 $EndComp
 $Comp
-L GND #PWR2
+L GND #PWR01
 U 1 1 536E9B70
 P 4725 2600
-F 0 "#PWR2" H 4725 2600 30  0001 C CNN
+F 0 "#PWR01" H 4725 2600 30  0001 C CNN
 F 1 "GND" H 4725 2530 30  0001 C CNN
 F 2 "" H 4725 2600 60  0000 C CNN
@@
 Connection ~ 4725 2525
 $Comp
-L GND #PWR5
+L GND #PWR02
 U 1 1 536E9BA0
 P 4625 3675
-F 0 "#PWR5" H 4625 3675 30  0001 C CNN
+F 0 "#PWR02" H 4625 3675 30  0001 C CNN
 F 1 "GND" H 4625 3605 30  0001 C CNN
 F 2 "" H 4625 3675 60  0000 C CNN
@@
 Connection ~ 4625 3600
 $Comp
-L GND #PWR8
+L GND #PWR03
 U 1 1 536E9BE2
 P 4725 4775
-F 0 "#PWR8" H 4725 4775 30  0001 C CNN
+F 0 "#PWR03" H 4725 4775 30  0001 C CNN
 F 1 "GND" H 4725 4705 30  0001 C CNN
 F 2 "" H 4725 4775 60  0000 C CNN
@@
 	3100 1825 4875 1825
 $Comp
-L +12V #PWR1
+L +12V #PWR04
 U 1 1 536E9C72
 P 5925 1675
-F 0 "#PWR1" H 5925 1625 20  0001 C CNN
+F 0 "#PWR04" H 5925 1625 20  0001 C CNN
 F 1 "+12V" H 5925 1775 30  0000 C CNN
 F 2 "" H 5925 1675 60  0000 C CNN
@@
 	5925 1825 5725 1825
 $Comp
-L +12V #PWR3
+L +12V #PWR05
 U 1 1 536E9CB2
 P 5950 2825
-F 0 "#PWR3" H 5950 2775 20  0001 C CNN
+F 0 "#PWR05" H 5950 2775 20  0001 C CNN
 F 1 "+12V" H 5950 2925 30  0000 C CNN
 F 2 "" H 5950 2825 60  0000 C CNN
@@
 	5950 2900 5725 2900
 $Comp
-L +12V #PWR7
+L +12V #PWR06
 U 1 1 536E9CE2
 P 5925 3950
-F 0 "#PWR7" H 5925 3900 20  0001 C CNN
+F 0 "#PWR06" H 5925 3900 20  0001 C CNN
 F 1 "+12V" H 5925 4050 30  0000 C CNN
 F 2 "" H 5925 3950 60  0000 C CNN
@@
 Connection ~ 7500 5250
 $Comp
-L GND #PWR9
+L GND #PWR07
 U 1 1 536EA382
 P 6825 5925
-F 0 "#PWR9" H 6825 5925 30  0001 C CNN
+F 0 "#PWR07" H 6825 5925 30  0001 C CNN
 F 1 "GND" H 6825 5855 30  0001 C CNN
 F 2 "" H 6825 5925 60  0000 C CNN
@@
 $EndComp
 $Comp
-L GND #PWR10
+L GND #PWR08
 U 1 1 536EA39F
 P 7175 5925
-F 0 "#PWR10" H 7175 5925 30  0001 C CNN
+F 0 "#PWR08" H 7175 5925 30  0001 C CNN
 F 1 "GND" H 7175 5855 30  0001 C CNN
 F 2 "" H 7175 5925 60  0000 C CNN
@@
 $EndComp
 $Comp
-L GND #PWR11
+L GND #PWR09
 U 1 1 536EA3BC
 P 7500 5925
-F 0 "#PWR11" H 7500 5925 30  0001 C CNN
+F 0 "#PWR09" H 7500 5925 30  0001 C CNN
 F 1 "GND" H 7500 5855 30  0001 C CNN
 F 2 "" H 7500 5925 60  0000 C CNN
@@
 Wire Wire Line
 	7500 5825 7500 5925
-$Comp
-L CONN_9 P1
-U 1 1 536EA4F9
+Wire Wire Line
+	2450 3100 2700 3100
+Wire Wire Line
+	2525 3100 2525 3300
+Wire Wire Line
+	2525 3200 2450 3200
+Wire Wire Line
+	2525 3300 2450 3300
+Connection ~ 2525 3200
+$Comp
+L GND #PWR010
+U 1 1 536EA780
+P 2700 3150
+F 0 "#PWR010" H 2700 3150 30  0001 C CNN
+F 1 "GND" H 2700 3080 30  0001 C CNN
+F 2 "" H 2700 3150 60  0000 C CNN
+F 3 "" H 2700 3150 60  0000 C CNN
+	1    2700 3150
+	1    0    0    -1
+$EndComp
+Wire Wire Line
+	2700 3100 2700 3150
+Connection ~ 2525 3100
+$Comp
+L +12V #PWR011
+U 1 1 536EA7F1
+P 2750 3950
+F 0 "#PWR011" H 2750 3900 20  0001 C CNN
+F 1 "+12V" H 2750 4050 30  0000 C CNN
+F 2 "" H 2750 3950 60  0000 C CNN
+F 3 "" H 2750 3950 60  0000 C CNN
+	1    2750 3950
+	1    0    0    -1
+$EndComp
+Wire Wire Line
+	2450 3950 2750 3950
+Wire Wire Line
+	2525 3750 2525 3950
+Wire Wire Line
+	2525 3850 2450 3850
+Connection ~ 2525 3950
+Wire Wire Line
+	2525 3750 2450 3750
+Connection ~ 2525 3850
+Wire Wire Line
+	2450 3425 3100 3425
+Wire Wire Line
+	3100 3425 3100 1825
+Wire Wire Line
+	3725 2900 3725 3525
+Wire Wire Line
+	3725 3525 2450 3525
+Wire Wire Line
+	2450 3625 3350 3625
+Wire Wire Line
+	3350 3625 3350 4025
+$Comp
+L CONN_3 K1
+U 1 1 536EA049
+P 2100 3200
+F 0 "K1" V 2050 3200 50  0000 C CNN
+F 1 "CONN_GND" V 2250 3250 40  0000 C CNN
+F 2 "" H 2100 3200 60  0000 C CNN
+F 3 "" H 2100 3200 60  0000 C CNN
+	1    2100 3200
+	-1   0    0    -1
+$EndComp
+$Comp
+L CONN_3 K2
+U 1 1 536EA083
 P 2100 3525
-F 0 "P1" V 2050 3525 60  0000 C CNN
-F 1 "CONN_9" V 2150 3525 60  0000 C CNN
+F 0 "K2" V 2050 3525 50  0000 C CNN
+F 1 "CONN_LEDS" V 2250 3525 40  0000 C CNN
 F 2 "" H 2100 3525 60  0000 C CNN
 F 3 "" H 2100 3525 60  0000 C CNN
@@
 	-1   0    0    -1
 $EndComp
-Wire Wire Line
-	2450 3125 2700 3125
-Wire Wire Line
-	2525 3125 2525 3325
-Wire Wire Line
-	2525 3225 2450 3225
-Wire Wire Line
-	2525 3325 2450 3325
-Connection ~ 2525 3225
-$Comp
-L GND #PWR4
-U 1 1 536EA780
-P 2700 3175
-F 0 "#PWR4" H 2700 3175 30  0001 C CNN
-F 1 "GND" H 2700 3105 30  0001 C CNN
-F 2 "" H 2700 3175 60  0000 C CNN
-F 3 "" H 2700 3175 60  0000 C CNN
-	1    2700 3175
-	1    0    0    -1
-$EndComp
-Wire Wire Line
-	2700 3125 2700 3175
-Connection ~ 2525 3125
-$Comp
-L +12V #PWR6
-U 1 1 536EA7F1
-P 2750 3925
-F 0 "#PWR6" H 2750 3875 20  0001 C CNN
-F 1 "+12V" H 2750 4025 30  0000 C CNN
-F 2 "" H 2750 3925 60  0000 C CNN
-F 3 "" H 2750 3925 60  0000 C CNN
-	1    2750 3925
-	1    0    0    -1
-$EndComp
-Wire Wire Line
-	2450 3925 2750 3925
-Wire Wire Line
-	2525 3725 2525 3925
-Wire Wire Line
-	2525 3825 2450 3825
-Connection ~ 2525 3925
-Wire Wire Line
-	2525 3725 2450 3725
-Connection ~ 2525 3825
-Wire Wire Line
-	2450 3425 3100 3425
-Wire Wire Line
-	3100 3425 3100 1825
-Wire Wire Line
-	3725 2900 3725 3525
-Wire Wire Line
-	3725 3525 2450 3525
-Wire Wire Line
-	2450 3625 3350 3625
-Wire Wire Line
-	3350 3625 3350 4025
+$Comp
+L CONN_3 K3
+U 1 1 536EA0BA
+P 2100 3850
+F 0 "K3" V 2050 3850 50  0000 C CNN
+F 1 "CONN_12V" V 2250 3800 40  0000 C CNN
+F 2 "" H 2100 3850 60  0000 C CNN
+F 3 "" H 2100 3850 60  0000 C CNN
+	1    2100 3850
+	-1   0    0    -1
+$EndComp
 $EndSCHEMATC
