File: loraine/hardware/uplighter/uplighter.sch (KiCad schematic (older format))
At the start: 17 parts, among them CON1 BARREL_JACK, K1 CONN_3, K2 CONN_3, K3 CONN_3, P1 POWER_THRU, P2 POWER, P3 SOLDER_PAD, U1 TL4242, U2 TL4242, U3 TL4242

Commit message: Nominally finished both PCBs
Parts:
- R1, R2, R3: value R -> 1R2
Connections:
- net GND: now also CON1.3
- no-connect marks 7 -> 6
Other:
- note added: "1W star, actual R=1.2\nfor I=0.148A\nR dissipation = 26mW"
- note added: "Nominal resistor dissipation is\n1W star: 60mW\n3W star: 27mW"
- note removed: "Resistor dissipation is\n1W star: 60mW\n3W star: 27mW"
Changed lines of the file:
@@
 P 5700 5600
 F 0 "R1" V 5780 5600 40  0000 C CNN
-F 1 "R" V 5707 5601 40  0000 C CNN
+F 1 "1R2" V 5707 5601 40  0000 C CNN
 F 2 "" V 5630 5600 30  0000 C CNN
 F 3 "" H 5700 5600 30  0000 C CNN
@@
 P 5900 5600
 F 0 "R2" V 5980 5600 40  0000 C CNN
-F 1 "R" V 5907 5601 40  0000 C CNN
+F 1 "1R2" V 5907 5601 40  0000 C CNN
 F 2 "" V 5830 5600 30  0000 C CNN
 F 3 "" H 5900 5600 30  0000 C CNN
@@
 P 6100 5600
 F 0 "R3" V 6180 5600 40  0000 C CNN
-F 1 "R" V 6107 5601 40  0000 C CNN
+F 1 "1R2" V 6107 5601 40  0000 C CNN
 F 2 "" V 6030 5600 30  0000 C CNN
 F 3 "" H 6100 5600 30  0000 C CNN
@@
 	1    0    0    -1
 $EndComp
-Text Notes 6300 5450 0    60   ~ 0
+Text Notes 6275 5025 0    60   ~ 0
 These current sense resistors\nset the peak LED current.\nREF is held at 177mV nominal
-Text Notes 6300 5700 0    60   ~ 0
+Text Notes 6275 5275 0    60   ~ 0
 3W star wants I=0.35A R=0.51\n1W star wants I=0.15A R=1.18
-Text Notes 6300 6050 0    60   ~ 0
-Resistor dissipation is\n1W star: 60mW\n3W star: 27mW
+Text Notes 6275 5600 0    60   ~ 0
+Nominal resistor dissipation is\n1W star: 60mW\n3W star: 27mW
 $Comp
 L CONN_3 K1
@@
 REF_BLUE
 $Comp
-L GND #PWR7
+L GND #PWR01
 U 1 1 53790258
 P 5700 5900
-F 0 "#PWR7" H 5700 5900 30  0001 C CNN
+F 0 "#PWR01" H 5700 5900 30  0001 C CNN
 F 1 "GND" H 5700 5830 30  0001 C CNN
 F 2 "" H 5700 5900 60  0000 C CNN
@@
 $EndComp
 $Comp
-L GND #PWR8
+L GND #PWR02
 U 1 1 53790276
 P 5900 5900
-F 0 "#PWR8" H 5900 5900 30  0001 C CNN
+F 0 "#PWR02" H 5900 5900 30  0001 C CNN
 F 1 "GND" H 5900 5830 30  0001 C CNN
 F 2 "" H 5900 5900 60  0000 C CNN
@@
 $EndComp
 $Comp
-L GND #PWR11
+L GND #PWR03
 U 1 1 53790294
 P 6100 5900
-F 0 "#PWR11" H 6100 5900 30  0001 C CNN
+F 0 "#PWR03" H 6100 5900 30  0001 C CNN
 F 1 "GND" H 6100 5830 30  0001 C CNN
 F 2 "" H 6100 5900 60  0000 C CNN
@@
 $EndComp
 $Comp
-L GND #PWR1
+L GND #PWR04
 U 1 1 537904E9
 P 2500 2200
-F 0 "#PWR1" H 2500 2200 30  0001 C CNN
+F 0 "#PWR04" H 2500 2200 30  0001 C CNN
 F 1 "GND" H 2500 2130 30  0001 C CNN
 F 2 "" H 2500 2200 60  0000 C CNN
@@
 $EndComp
 $Comp
-L GND #PWR2
+L GND #PWR05
 U 1 1 537905EA
 P 2500 4100
-F 0 "#PWR2" H 2500 4100 30  0001 C CNN
+F 0 "#PWR05" H 2500 4100 30  0001 C CNN
 F 1 "GND" H 2500 4030 30  0001 C CNN
 F 2 "" H 2500 4100 60  0000 C CNN
@@
 $EndComp
 $Comp
-L GND #PWR3
+L GND #PWR06
 U 1 1 53790784
 P 2500 6000
-F 0 "#PWR3" H 2500 6000 30  0001 C CNN
+F 0 "#PWR06" H 2500 6000 30  0001 C CNN
 F 1 "GND" H 2500 5930 30  0001 C CNN
 F 2 "" H 2500 6000 60  0000 C CNN
@@
 $EndComp
 $Comp
-L GND #PWR10
+L GND #PWR07
 U 1 1 537A6CCB
 P 6100 2350
-F 0 "#PWR10" H 6100 2350 30  0001 C CNN
+F 0 "#PWR07" H 6100 2350 30  0001 C CNN
 F 1 "GND" H 6100 2280 30  0001 C CNN
 F 2 "" H 6100 2350 60  0000 C CNN
@@
 	-1   0    0    1
 $EndComp
-NoConn ~ 8325 1625
-$Comp
-L +5V #PWR4
+$Comp
+L +5V #PWR08
 U 1 1 53CD6A41
 P 2650 1150
-F 0 "#PWR4" H 2650 1240 20  0001 C CNN
+F 0 "#PWR08" H 2650 1240 20  0001 C CNN
 F 1 "+5V" H 2650 1240 30  0000 C CNN
 F 2 "" H 2650 1150 60  0000 C CNN
@@
 $EndComp
 $Comp
-L +5V #PWR5
+L +5V #PWR09
 U 1 1 53CD6ACD
 P 2650 3050
-F 0 "#PWR5" H 2650 3140 20  0001 C CNN
+F 0 "#PWR09" H 2650 3140 20  0001 C CNN
 F 1 "+5V" H 2650 3140 30  0000 C CNN
 F 2 "" H 2650 3050 60  0000 C CNN
@@
 $EndComp
 $Comp
-L +5V #PWR6
+L +5V #PWR010
 U 1 1 53CD6B6A
 P 2650 4950
-F 0 "#PWR6" H 2650 5040 20  0001 C CNN
+F 0 "#PWR010" H 2650 5040 20  0001 C CNN
 F 1 "+5V" H 2650 5040 30  0000 C CNN
 F 2 "" H 2650 4950 60  0000 C CNN
@@
 $EndComp
 $Comp
-L +5V #PWR9
+L +5V #PWR011
 U 1 1 53CD6C4B
 P 6100 1650
-F 0 "#PWR9" H 6100 1740 20  0001 C CNN
+F 0 "#PWR011" H 6100 1740 20  0001 C CNN
 F 1 "+5V" H 6100 1740 30  0000 C CNN
 F 2 "" H 6100 1650 60  0000 C CNN
@@
 $EndComp
 $Comp
-L +5V #PWR12
+L +5V #PWR012
 U 1 1 53CD7008
 P 8950 1475
-F 0 "#PWR12" H 8950 1565 20  0001 C CNN
+F 0 "#PWR012" H 8950 1565 20  0001 C CNN
 F 1 "+5V" H 8950 1565 30  0000 C CNN
 F 2 "" H 8950 1475 60  0000 C CNN
@@
 $EndComp
 $Comp
-L GND #PWR13
+L GND #PWR013
 U 1 1 53CD70A7
 P 8950 1775
-F 0 "#PWR13" H 8950 1775 30  0001 C CNN
+F 0 "#PWR013" H 8950 1775 30  0001 C CNN
 F 1 "GND" H 8950 1705 30  0001 C CNN
 F 2 "" H 8950 1775 60  0000 C CNN
@@
 NoConn ~ 2300 3450
 NoConn ~ 2300 5350
+Text Notes 6275 5925 0    60   ~ 0
+1W star, actual R=1.2\nfor I=0.148A\nR dissipation = 26mW
+Wire Wire Line
+	8325 1625 8425 1625
+Wire Wire Line
+	8425 1625 8425 1725
+Connection ~ 8425 1725
+$Comp
+L PWR_FLAG #FLG014
+U 1 1 53D68080
+P 2175 1200
+F 0 "#FLG014" H 2175 1295 30  0001 C CNN
+F 1 "PWR_FLAG" H 2175 1380 30  0000 C CNN
+F 2 "" H 2175 1200 60  0000 C CNN
+F 3 "" H 2175 1200 60  0000 C CNN
+	1    2175 1200
+	1    0    0    -1
+$EndComp
+Connection ~ 2175 1200
+$Comp
+L PWR_FLAG #FLG015
+U 1 1 53D685F8
+P 1975 1750
+F 0 "#FLG015" H 1975 1845 30  0001 C CNN
+F 1 "PWR_FLAG" H 1975 1930 30  0000 C CNN
+F 2 "" H 1975 1750 60  0000 C CNN
+F 3 "" H 1975 1750 60  0000 C CNN
+	1    1975 1750
+	0    -1   -1   0
+$EndComp
+Wire Wire Line
+	1975 1750 2025 1750
+Wire Wire Line
+	2025 1750 2025 1650
+Connection ~ 2025 1650
 $EndSCHEMATC
