File: loraine/hardware/node/loraine_node.kicad_pcb (KiCad board)
At the start: 2 copper layers, 50 x 50 mm, 45 parts, among them CON1 BARREL_JACK, IC1 ATTINY2313A-S, K1 LED1, K2 LED2, K3 LED3, P1 POWER_THRU, P2 POWER, P3 SOLDER_PAD, P4 BUS, P5 BUS_THRU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

Commit message: Prettified PCB
Parts:
- added G***: LOGO, lorraine:lorraine, B.Cu at (125.0, 130.4)
- moved P5 2.17 mm to (110.4, 146.8)
- moved C4 1.09 mm to (107.6, 142.9), turned to 0 degrees
- moved P4 1.02 mm to (103.4, 146.1)
- moved P1 0.89 mm to (103.1, 104.1)
- moved P2 0.13 mm to (108.7, 102.9)
Connections:
- net /MISO renamed /LED6
- net Net-(IC1-Pad12) renamed /LED0
- net Net-(IC1-Pad14) renamed /LED2
- net Net-(P4-Pad1) renamed /A
- net Net-(P4-Pad2) renamed /B
- net Net-(P7-Pad10) renamed /CH4
- net Net-(P7-Pad12) renamed /CH5
- net Net-(P7-Pad14) renamed /CH6
- net Net-(P7-Pad16) renamed /CH7
- net Net-(P7-Pad2) renamed /CH0
- net Net-(P7-Pad4) renamed /CH1
- net Net-(P7-Pad6) renamed /CH2
- net Net-(P7-Pad8) renamed /CH3
Routing:
- net GND: track 47.1 -> 52.9 mm, vias 22 -> 23
- net /LED0: track 41.7 -> 44.5 mm
- net +5V: track 134.7 -> 136.7 mm
- net Net-(C2-Pad1): track 24.3 -> 22.6 mm
- net Net-(C1-Pad1): track 16.4 -> 14.9 mm
- net /LED2: track 48.5 -> 49.7 mm
- net VIN: track 118.7 -> 117.9 mm
- net /B: track 12.0 -> 12.7 mm
- net /CH1: track 16.9 -> 17.6 mm
- added copper zone on F.Cu, net GND
Other:
- board text added: ""She looked as beautiful as ever""
- board text added: "+"
- board text added: "0"
- board text added: "1"
- board text added: "2"
- board text added: "3"
- board text added: "4"
- board text added: "5"
- board text added: "5V"
- board text added: "6"
- board text added: "7"
- board text added: "A"
- board text added: "B"
- board text added: "CH0"
- board text added: "CH2"
- board text added: "CH6"
- board text added: "DATA"
- board text added: "DAVID TURNER ADAM GREIG"
- board text added: "GND"
- board text added: "LORAINE"
- board text added: "MISO"
- board text added: "MOSI"
- board text added: "RESET"
- board text added: "SCK"

Commit message: Adam's changes and gerbils
Parts:
- C4: value 0.1uF -> 0.1u
- moved P2 0.63 mm to (108.7, 103.5)
- moved P1 0.25 mm to (103.4, 104.1), turned to 270 degrees
- turned P5 to 0 degrees
Connections:
- CON1 pad 3: (no net) -> GND
Routing:
- net /B: track 12.7 -> 16.6 mm
- net GND: track 52.9 -> 55.0 mm
- net /A: track 19.8 -> 18.2 mm
- net /LED2: track 49.7 -> 51.2 mm
- net /RESET: track 9.81 -> 11.0 mm
- net /LED6: track 49.6 -> 50.7 mm
- net +5V: track 136.7 -> 136.0 mm
- net VIN: track 117.9 -> 117.3 mm
Other:
- rule via_min_drill: 0.508 -> 0.6
- rule via_min_size: 1.26 -> 1.2

Commit message: Added revision and date to silk
Other:
- board text added: "2014-07-27"
- board text added: "r1"
